Commit message: addition of description and simulation stuff

File: arm_description/models/al5d_macro.urdf.xacro (robot description, xacro)
@@ -11,5 +11,4 @@
   <property name="link4_length" value="0.032" />
   <property name="gripper_offset" value="0.016" />
-  <!--TODO add the additional wrist joint and link for the al5d 5DOF version-->
   <xacro:macro name="lynxmotion_al5d" params="prefix parent_link *origin">
     <!-- attach -->
@@ -181,11 +180,64 @@
       <limit lower="-${M_PI/2}" upper="${M_PI/2}" effort="0" velocity="6.98"/>
     </joint>
-    <joint name="${prefix}gripper" type="fixed">
+    <joint name="${prefix}gripper" type="revolute">
       <origin xyz="${link4_length + gripper_offset} 0 0" rpy="0 0 0"/>
       <parent link="${prefix}link_4"/>
       <child link="${prefix}gripper"/>
-      <axis xyz="0 0 1"/>
+      <axis xyz="1 0 0"/>
       <limit lower="-${M_PI/2}" upper="${M_PI/2}" effort="0" velocity="6.98"/>
     </joint>
+    <transmission name="${prefix}joint_1">
+      <type>transmission_interface/SimpleTransmission</type>
+      <joint name="${prefix}joint_1">
+        <hardwareInterface>hardware_interface/PositionJointInterface</hardwareInterface>
+      </joint>
+      <actuator name="motor1">
+        <hardwareInterface>hardware_interface/PositionJointInterface</hardwareInterface>
+        <mechanicalReduction>1</mechanicalReduction>
+      </actuator>
+    </transmission>
+    <transmission name="${prefix}joint_2">
+      <type>transmission_interface/SimpleTransmission</type>
+      <joint name="${prefix}joint_2">
+        <hardwareInterface>hardware_interface/PositionJointInterface</hardwareInterface>
+      </joint>
+      <actuator name="motor2">
+        <hardwareInterface>hardware_interface/PositionJointInterface</hardwareInterface>
+        <mechanicalReduction>1</mechanicalReduction>
+      </actuator>
+    </transmission>
+    <transmission name="${prefix}joint_3">
+      <type>transmission_interface/SimpleTransmission</type>
+      <joint name="${prefix}joint_3">
+        <hardwareInterface>hardware_interface/PositionJointInterface</hardwareInterface>
+      </joint>
+      <actuator name="motor3">
+        <hardwareInterface>hardware_interface/PositionJointInterface</hardwareInterface>
+        <mechanicalReduction>1</mechanicalReduction>
+      </actuator>
+    </transmission>
+    <transmission name="${prefix}joint_4">
+      <type>transmission_interface/SimpleTransmission</type>
+      <joint name="${prefix}joint_4">
+        <hardwareInterface>hardware_interface/PositionJointInterface</hardwareInterface>
+      </joint>
+      <actuator name="motor4">
+        <hardwareInterface>hardware_interface/PositionJointInterface</hardwareInterface>
+        <mechanicalReduction>1</mechanicalReduction>
+      </actuator>
+    </transmission>
+    <transmission name="${prefix}gripper">
+      <type>transmission_interface/SimpleTransmission</type>
+      <joint name="${prefix}gripper">
+        <hardwareInterface>hardware_interface/PositionJointInterface</hardwareInterface>
+      </joint>
+      <actuator name="motor5">
+        <hardwareInterface>hardware_interface/PositionJointInterface</hardwareInterface>
+        <mechanicalReduction>1</mechanicalReduction>
+      </actuator>
+    </transmission>
+    <gazebo>
+      <plugin name="control" filename="libgazebo_ros_control.so"/>
+    </gazebo>
   </xacro:macro>
 </robot>

Commit message: Initial control using RVIZ and moveit. Missed a major joint so control is limited to a 2D plane of the arm.

File: arm_description/models/al5d_macro.urdf.xacro (robot description, xacro)
@@ -11,5 +11,5 @@
   <property name="link4_length" value="0.032" />
   <property name="gripper_offset" value="0.016" />
-  <xacro:macro name="lynxmotion_al5d" params="prefix parent_link *origin">
+  <xacro:macro name="lynxmotion_al5d" params="prefix parent_link rate:=50 *origin">
     <!-- attach -->
     <joint name="arm_base_joint" type="fixed">
@@ -239,4 +239,8 @@
     <gazebo>
       <plugin name="control" filename="libgazebo_ros_control.so"/>
+      <plugin name="joint_state_publisher" filename="libgazebo_ros_joint_state_publisher.so">
+        <jointName>${prefix}joint_1, ${prefix}joint_2, ${prefix}joint_3, ${prefix}joint_4, ${prefix}gripper</jointName>
+        <updateRate>${rate}</updateRate>
+      </plugin>
     </gazebo>
   </xacro:macro>

Commit message: Some general code cleanup

File: arm_description/models/al5d_macro.urdf.xacro (robot description, xacro)
@@ -2,17 +2,17 @@
 <robot xmlns:xacro="http://ros.org/wiki/xacro">
   <xacro:property name="M_PI" value="3.14159"/>
-  <property name="base_height" value="0.043" />
-  <property name="base_radius" value="0.048" />
-  <property name="link1_height" value="0.006" />
-  <property name="link1_radius" value="0.048" />
-  <property name="link2_offset" value="0.022" />
-  <property name="link2_length" value="0.14605" />
-  <property name="link3_length" value="0.187325" />
-  <property name="link4_length" value="0.032" />
-  <property name="gripper_offset" value="0.016" />
+  <xacro:property name="base_height" value="0.043" />
+  <xacro:property name="base_radius" value="0.048" />
+  <xacro:property name="link1_height" value="0.006" />
+  <xacro:property name="link1_radius" value="0.048" />
+  <xacro:property name="link2_offset" value="0.022" />
+  <xacro:property name="link2_length" value="0.14605" />
+  <xacro:property name="link3_length" value="0.187325" />
+  <xacro:property name="link4_length" value="0.032" />
+  <xacro:property name="gripper_offset" value="0.016" />
   <xacro:macro name="lynxmotion_al5d" params="prefix parent_link rate:=50 *origin">
     <!-- attach -->
     <joint name="arm_base_joint" type="fixed">
-      <insert_block name="origin" />
+      <xacro:insert_block name="origin" />
       <parent link="${parent_link}"/>
       <child link="${prefix}base_link" />
